File: usb_uart.sch (KiCad schematic (older format))
At the start: 23 parts, among them J1 Conn_01x03_Female, J2 USB_B, J3 Conn_01x03_Female, Q1 Q_NMOS_DGS, Q2 Q_NMOS_DGS, U1 FT230FX

Commit message: First draft pcb
TODO: fix the rts/cts signals
Parts:
- removed J1, J3: Conn_01x03_Female, symbol Connector:Conn_01x03_Female
- removed Q1, Q2: Q_NMOS_DGS, symbol device:Q_NMOS_DGS
- added J1, J3: Conn_01x04_Female, Connector_PinHeader_2.54mm:PinHeader_1x04_P2.54mm_Horizontal, symbol Connector:Conn_01x04_Female
- added Q1, Q2: DMG2302UK, Package_TO_SOT_SMD:SOT-23_Handsoldering, symbol device:Q_NMOS_GSD
- added R9: 0, Resistors_SMD:R_0805_HandSoldering, symbol device:R
- C1, C2, C3, C4, C5, C6: footprint (none) -> Capacitors_SMD:C_0603_HandSoldering
- D1, D2: footprint (none) -> LED_SMD:LED_1206_3216Metric_Pad1.07x1.80mm_HandSolder
- F1: footprint (none) -> Fuse:Fuse_1206_3216Metric_Pad1.24x1.80mm_HandSolder
- J2: footprint (none) -> Connector_USB:USB_B_Horizontal
- R1, R2, R3, R4, R5, R6, R7, R8: footprint (none) -> Resistors_SMD:R_0805_HandSoldering
- U1: footprint (none) -> Package_SSOP:SSOP-16_3.9x4.9mm_P0.635mm
Connections:
- wire segments 75 -> 78
